File: jantteri-lora/_autosave-jantteri-lora.sch (KiCad schematic (older format))
At the start: 0 parts

Commit message: jantteri-lora work
Parts:
- added D? (x2): D_Small, symbol Device:D_Small
- added FB?: GZ2012D101TF, Inductor_SMD:L_0805_2012Metric, symbol Device:Ferrite_Bead
- added U?: lora-mod, symbol voja-lib:lora-mod
Connections:
- net labels added: 5V-IN, DATA1, DATA10, DATA11, DATA12, DATA13, DATA14, DATA15, DATA16, DATA2, DATA3, DATA4, DATA5, DATA6, DATA7, DATA8, DATA9, OUTPUT_SCL, OUTPUT_SDA, USB-5V
- wire segments 17 -> 24
Changed lines of the file:
@@
 $EndDescr
-$Sheet
-S 2350 1450 550  300
-U 611583F8
-F0 "polarity-protection" 50
-F1 "polarity-protection.sch" 50
-F2 "VIN" I L 2350 1550 50
-F3 "VOUT" I R 2900 1550 50
-F4 "GND" I L 2350 1650 50
-$EndSheet
 $Sheet
 S 3650 1450 550  400
@@
 $EndSheet
 $Comp
-L power:+3V3 #PWR?
+L power:+3V3 #PWR0101
 U 1 1 61143103
 P 5850 1850
-F 0 "#PWR?" H 5850 1700 50  0001 C CNN
+F 0 "#PWR0101" H 5850 1700 50  0001 C CNN
 F 1 "+3V3" H 5865 2023 50  0000 C CNN
 F 2 "" H 5850 1850 50  0001 C CNN
@@
 $EndComp
 $Comp
-L power:GND #PWR?
+L power:GND #PWR0102
 U 1 1 611435CD
 P 5850 1950
-F 0 "#PWR?" H 5850 1700 50  0001 C CNN
+F 0 "#PWR0102" H 5850 1700 50  0001 C CNN
 F 1 "GND" H 5855 1777 50  0000 C CNN
 F 2 "" H 5850 1950 50  0001 C CNN
@@
 	6100 3100 5900 3100
 $Comp
-L power:GND #PWR?
+L power:GND #PWR0103
 U 1 1 611483EC
 P 5050 2500
-F 0 "#PWR?" H 5050 2250 50  0001 C CNN
+F 0 "#PWR0103" H 5050 2250 50  0001 C CNN
 F 1 "GND" H 5055 2327 50  0000 C CNN
 F 2 "" H 5050 2500 50  0001 C CNN
@@
 $EndComp
 $Comp
-L power:GND #PWR?
+L power:GND #PWR0104
 U 1 1 61148B21
 P 5050 3150
-F 0 "#PWR?" H 5050 2900 50  0001 C CNN
+F 0 "#PWR0104" H 5050 2900 50  0001 C CNN
 F 1 "GND" H 5055 2977 50  0000 C CNN
 F 2 "" H 5050 3150 50  0001 C CNN
@@
 $EndComp
 $Comp
-L power:+3V3 #PWR?
+L power:+3V3 #PWR0105
 U 1 1 61148EAA
 P 5050 2400
-F 0 "#PWR?" H 5050 2250 50  0001 C CNN
+F 0 "#PWR0105" H 5050 2250 50  0001 C CNN
 F 1 "+3V3" H 5065 2573 50  0000 C CNN
 F 2 "" H 5050 2400 50  0001 C CNN
@@
 	5250 2400 5050 2400
 $Comp
-L power:+3V3 #PWR?
+L power:+3V3 #PWR0106
 U 1 1 6114B431
 P 8050 1850
-F 0 "#PWR?" H 8050 1700 50  0001 C CNN
+F 0 "#PWR0106" H 8050 1700 50  0001 C CNN
 F 1 "+3V3" H 8065 2023 50  0000 C CNN
 F 2 "" H 8050 1850 50  0001 C CNN
@@
 $EndComp
 $Comp
-L power:GND #PWR?
+L power:GND #PWR0107
 U 1 1 6114B78E
 P 8050 1950
-F 0 "#PWR?" H 8050 1700 50  0001 C CNN
+F 0 "#PWR0107" H 8050 1700 50  0001 C CNN
 F 1 "GND" H 8055 1777 50  0000 C CNN
 F 2 "" H 8050 1950 50  0001 C CNN
@@
 	2900 1550 3650 1550
 $Comp
-L power:GND #PWR?
+L power:GND #PWR0108
 U 1 1 6114C811
 P 3550 1650
-F 0 "#PWR?" H 3550 1400 50  0001 C CNN
+F 0 "#PWR0108" H 3550 1400 50  0001 C CNN
 F 1 "GND" H 3555 1477 50  0000 C CNN
 F 2 "" H 3550 1650 50  0001 C CNN
@@
 	1    0    0    -1
 $EndComp
-$Comp
-L power:GND #PWR?
-U 1 1 6114CC51
-P 2250 1650
-F 0 "#PWR?" H 2250 1400 50  0001 C CNN
-F 1 "GND" H 2255 1477 50  0000 C CNN
-F 2 "" H 2250 1650 50  0001 C CNN
-F 3 "" H 2250 1650 50  0001 C CNN
-	1    2250 1650
-	1    0    0    -1
-$EndComp
-Wire Wire Line
-	2250 1650 2350 1650
 Wire Wire Line
 	3550 1650 3650 1650
 $Comp
-L power:+3V3 #PWR?
+L power:+3V3 #PWR0110
 U 1 1 6114D52E
 P 4550 1550
-F 0 "#PWR?" H 4550 1400 50  0001 C CNN
+F 0 "#PWR0110" H 4550 1400 50  0001 C CNN
 F 1 "+3V3" H 4565 1723 50  0000 C CNN
 F 2 "" H 4550 1550 50  0001 C CNN
@@
 Wire Wire Line
 	5050 3100 5050 3150
+Text GLabel 5250 3000 0    50   Input ~ 0
+USB-5V
+$Comp
+L Device:Ferrite_Bead FB?
+U 1 1 6115E9C4
+P 2750 1550
+AR Path="/611583F8/6115E9C4" Ref="FB?"  Part="1"
+AR Path="/6115E9C4" Ref="FB?"  Part="1"
+F 0 "FB?" V 2476 1550 50  0000 C CNN
+F 1 "GZ2012D101TF" V 2567 1550 50  0000 C CNN
+F 2 "Inductor_SMD:L_0805_2012Metric" V 2680 1550 50  0001 C CNN
+F 3 "~" H 2750 1550 50  0001 C CNN
+F 4 "C1015" V 2750 1550 50  0001 C CNN "LCSC"
+	1    2750 1550
+	0    1    1    0
+$EndComp
+Text GLabel 1600 1350 0    50   Input ~ 0
+USB-5V
+Text GLabel 1550 1750 0    50   Input ~ 0
+5V-IN
+$Comp
+L Device:D_Small D?
+U 1 1 61160523
+P 1950 1350
+F 0 "D?" H 1950 1143 50  0000 C CNN
+F 1 "D_Small" H 1950 1234 50  0000 C CNN
+F 2 "" V 1950 1350 50  0001 C CNN
+F 3 "~" V 1950 1350 50  0001 C CNN
+	1    1950 1350
+	-1   0    0    1
+$EndComp
+$Comp
+L Device:D_Small D?
+U 1 1 61161104
+P 1950 1750
+F 0 "D?" H 1950 1543 50  0000 C CNN
+F 1 "D_Small" H 1950 1634 50  0000 C CNN
+F 2 "" V 1950 1750 50  0001 C CNN
+F 3 "~" V 1950 1750 50  0001 C CNN
+	1    1950 1750
+	-1   0    0    1
+$EndComp
+Wire Wire Line
+	1600 1350 1850 1350
+Wire Wire Line
+	1550 1750 1850 1750
+Wire Wire Line
+	2050 1750 2350 1750
+Wire Wire Line
+	2350 1750 2350 1550
+Wire Wire Line
+	2350 1550 2600 1550
+Wire Wire Line
+	2050 1350 2350 1350
+Wire Wire Line
+	2350 1350 2350 1550
+Connection ~ 2350 1550
+Text GLabel 3000 3000 2    50   Input ~ 0
+5V-IN
+$Comp
+L power:GND #PWR?
+U 1 1 61169965
+P 3500 3100
+F 0 "#PWR?" H 3500 2850 50  0001 C CNN
+F 1 "GND" H 3505 2927 50  0000 C CNN
+F 2 "" H 3500 3100 50  0001 C CNN
+F 3 "" H 3500 3100 50  0001 C CNN
+	1    3500 3100
+	1    0    0    -1
+$EndComp
+Wire Wire Line
+	3000 3100 3500 3100
+Text GLabel 2050 3000 0    50   Input ~ 0
+OUTPUT_SDA
+Text GLabel 2050 3100 0    50   Input ~ 0
+OUTPUT_SCL
+Text GLabel 2050 3200 0    50   Input ~ 0
+DATA1
+$Comp
+L voja-lib:lora-mod U?
+U 1 1 61170943
+P 2550 3350
+F 0 "U?" H 2525 3925 50  0000 C CNN
+F 1 "lora-mod" H 2525 3834 50  0000 C CNN
+F 2 "" H 2550 3350 50  0001 C CNN
+F 3 "" H 2550 3350 50  0001 C CNN
+	1    2550 3350
+	1    0    0    -1
+$EndComp
+Text GLabel 2050 3300 0    50   Input ~ 0
+DATA2
+Text GLabel 2050 3400 0    50   Input ~ 0
+DATA3
+Text GLabel 2050 3500 0    50   Input ~ 0
+DATA4
+Text GLabel 2050 3600 0    50   Input ~ 0
+DATA5
+Text GLabel 2050 3700 0    50   Input ~ 0
+DATA6
+Text GLabel 2050 3800 0    50   Input ~ 0
+DATA7
+Text GLabel 2050 3900 0    50   Input ~ 0
+DATA8
+Text GLabel 3000 3200 2    50   Input ~ 0
+DATA9
+Text GLabel 3000 3300 2    50   Input ~ 0
+DATA10
+Text GLabel 3000 3400 2    50   Input ~ 0
+DATA11
+Text GLabel 3000 3500 2    50   Input ~ 0
+DATA12
+Text GLabel 3000 3600 2    50   Input ~ 0
+DATA13
+Text GLabel 3000 3700 2    50   Input ~ 0
+DATA14
+Text GLabel 3000 3800 2    50   Input ~ 0
+DATA15
+Text GLabel 3000 3900 2    50   Input ~ 0
+DATA16
 $EndSCHEMATC

Commit message: Lora PCB desging
Parts:
- removed D? (x2): D_Small, symbol Device:D_Small
- U1: renamed from U?; footprint (none) -> voja-footprints:lora-mod
- gave numbers to parts that had none: 1
Connections:
- net labels added: DBG_RX, DBG_TX, RFM_DIO0, RFM_NSS, RFM_RST, SPI1_MISO, SPI1_MOSI, SPI1_SCK
- wire segments 24 -> 28
- no-connect marks 1 -> 2
Other:
- note added: "5V-IN disables USB power input. If no 5V-IN connected, USB-5V is used"
- moved on the sheet: U1
