File: jantteri-lora/10pinARM.sch (KiCad schematic (older format))
At the start: 1 part, among them J2 SWD

Commit message: Lora-module v1
Parts:
- J2: footprint Connector_PinHeader_1.27mm:PinHeader_2x05_P1.27mm_Vertical_SMD -> Connector_PinHeader_1.27mm:PinHeader_2x05_P1.27mm_Horizontal
Changed lines of the file:
@@
 F 0 "J2" H 5250 4017 50  0000 C CNN
 F 1 "SWD" H 5250 3926 50  0000 C CNN
-F 2 "Connector_PinHeader_1.27mm:PinHeader_2x05_P1.27mm_Vertical_SMD" H 5200 3600 50  0001 C CNN
+F 2 "Connector_PinHeader_1.27mm:PinHeader_2x05_P1.27mm_Horizontal" H 5200 3600 50  0001 C CNN
 F 3 "~" H 5200 3600 50  0001 C CNN
 	1    5200 3600
