File: jantteri-lora/power_protect.sch (KiCad schematic (older format))
At the start: 5 parts, among them Q1 Si2319CDS, U4 AP2301

Commit message: Lora-module v1
Parts:
- Q1: value Si2319CDS -> IRLML6402TRPBF; LCSC C146287 -> C2593
- R3: renamed from 100K2; footprint (none) -> Resistor_SMD:R_0402_1005Metric; LCSC (none) -> C25741
- U4: symbol JLC_assembled:AP2301 -> jantteri-lora-rescue:AP2301-JLC_assembled
Changed lines of the file:
@@
 $Descr A4 11693 8268
 encoding utf-8
-Sheet 6 8
+Sheet 7 8
 Title ""
 Date ""
@@
 AR Path="/6118C146/61181872" Ref="C?"  Part="1"
 AR Path="/611A8D7A/61181872" Ref="C7"  Part="1"
-F 0 "C5" H 4342 2946 50  0000 L CNN
+F 0 "C7" H 4342 2946 50  0000 L CNN
 F 1 "100n" H 4342 2855 50  0000 L CNN
 F 2 "Capacitor_SMD:C_0603_1608Metric" H 4250 2900 50  0001 C CNN
@@
 AR Path="/6118C146/61186B4B" Ref="C?"  Part="1"
 AR Path="/611A8D7A/61186B4B" Ref="C8"  Part="1"
-F 0 "C6" H 5992 2946 50  0000 L CNN
+F 0 "C8" H 5992 2946 50  0000 L CNN
 F 1 "100n" H 5992 2855 50  0000 L CNN
 F 2 "Capacitor_SMD:C_0603_1608Metric" H 5900 2900 50  0001 C CNN
@@
 AR Path="/6117A90D/611A29C1" Ref="Q1"  Part="1"
 AR Path="/611A8D7A/611A29C1" Ref="Q2"  Part="1"
-F 0 "Q1" V 4042 2900 50  0000 C CNN
-F 1 "Si2319CDS" V 3951 2900 50  0000 C CNN
+F 0 "Q2" V 4042 2900 50  0000 C CNN
+F 1 "IRLML6402TRPBF" V 3951 2900 50  0000 C CNN
 F 2 "Package_TO_SOT_SMD:SOT-23" H 3900 2825 50  0001 L CIN
 F 3 "http://www.vishay.com/docs/66709/si2319cd.pdf" H 3700 2900 50  0001 L CNN
-F 4 "C146287" V 3700 2900 50  0001 C CNN "LCSC"
+F 4 "C2593" V 3700 2900 50  0001 C CNN "LCSC"
 	1    3700 2900
 	0    -1   -1   0
@@
 Connection ~ 4250 2800
 $Comp
-L Device:R_Small R?
+L Device:R_Small R3
 U 1 1 611A520B
 P 4600 3350
-AR Path="/6117A90D/611A520B" Ref="R?"  Part="1"
-AR Path="/611A8D7A/611A520B" Ref="100K2"  Part="1"
-F 0 "R?" H 4659 3396 50  0000 L CNN
+AR Path="/6117A90D/611A520B" Ref="R3"  Part="1"
+AR Path="/611A8D7A/611A520B" Ref="R4"  Part="1"
+F 0 "R4" H 4659 3396 50  0000 L CNN
 F 1 "100K" H 4659 3305 50  0000 L CNN
-F 2 "" H 4600 3350 50  0001 C CNN
+F 2 "Resistor_SMD:R_0402_1005Metric" H 4600 3350 50  0001 C CNN
 F 3 "~" H 4600 3350 50  0001 C CNN
+F 4 "C25741" H 4600 3350 50  0001 C CNN "LCSC"
 	1    4600 3350
 	1    0    0    -1
@@
 EN
 $Comp
-L JLC_assembled:AP2301 U4
+L jantteri-lora-rescue:AP2301-JLC_assembled U4
 U 1 1 61199B0A
 P 4950 2900
 AR Path="/6117A90D/61199B0A" Ref="U4"  Part="1"
 AR Path="/611A8D7A/61199B0A" Ref="U5"  Part="1"
-F 0 "U4" H 4975 3465 50  0000 C CNN
+AR Path="/61199B0A" Ref="U4"  Part="1"
+F 0 "U5" H 4975 3465 50  0000 C CNN
 F 1 "AP2301" H 4975 3374 50  0000 C CNN
 F 2 "Package_SO:MSOP-8-1EP_3x3mm_P0.65mm_EP1.68x1.88mm" H 5150 2500 50  0001 C CNN
