File: jantteri-lora/AMS1117-3.3.sch (KiCad schematic (older format))
At the start: 3 parts

Commit message: Lora PCB desging
Parts:
- gave numbers to parts that had none: 3
Changed lines of the file:
@@
 $Descr A4 11693 8268
 encoding utf-8
-Sheet 6 7
+Sheet 2 8
 Title ""
 Date ""
@@
 	4950 3300 5500 3300
 $Comp
-L Device:C_Small C?
+L Device:C_Small C2
 U 1 1 6115FB08
 P 5950 3200
-F 0 "C?" H 6042 3246 50  0000 L CNN
+F 0 "C2" H 6042 3246 50  0000 L CNN
 F 1 "10u" H 6042 3155 50  0000 L CNN
 F 2 "Capacitor_SMD:C_0805_2012Metric" H 5950 3200 50  0001 C CNN
@@
 $EndComp
 $Comp
-L Device:C_Small C?
+L Device:C_Small C1
 U 1 1 6115FB0F
 P 4950 3200
-F 0 "C?" H 5042 3246 50  0000 L CNN
+F 0 "C1" H 5042 3246 50  0000 L CNN
 F 1 "10u" H 5042 3155 50  0000 L CNN
 F 2 "Capacitor_SMD:C_0805_2012Metric" H 4950 3200 50  0001 C CNN
@@
 $EndComp
 $Comp
-L Regulator_Linear:AMS1117-3.3 U?
+L Regulator_Linear:AMS1117-3.3 U2
 U 1 1 6115FB16
 P 5500 2950
-F 0 "U?" H 5500 3192 50  0000 C CNN
+F 0 "U2" H 5500 3192 50  0000 C CNN
 F 1 "AMS1117-3.3" H 5500 3101 50  0000 C CNN
 F 2 "Package_TO_SOT_SMD:SOT-223-3_TabPin2" H 5500 3150 50  0001 C CNN
