File: jantteri-lora/STM32G030C8T6.sch (KiCad schematic (older format))
At the start: 14 parts

Commit message: Lora PCB desging
Parts:
- U6: renamed from U?; footprint (none) -> Package_QFP:LQFP-48_7x7mm_P0.5mm
- gave numbers to parts that had none: 13
Connections:
- net DBG_RX renamed PA10
- net DBG_TX renamed PA9
Changed lines of the file:
@@
 $Descr A4 11693 8268
 encoding utf-8
-Sheet 5 7
+Sheet 3 8
 Title ""
 Date ""
@@
 	3400 2350 3900 2350
 $Comp
-L Device:R_Small R?
+L Device:R_Small R2
 U 1 1 61169DFC
 P 7250 2250
-F 0 "R?" V 7054 2250 50  0000 C CNN
+F 0 "R2" V 7054 2250 50  0000 C CNN
 F 1 "47" V 7145 2250 50  0000 C CNN
 F 2 "Resistor_SMD:R_0402_1005Metric" H 7250 2250 50  0001 C CNN
@@
 $EndComp
 $Comp
-L Device:C_Small C?
+L Device:C_Small C17
 U 1 1 61169E03
 P 7000 2550
-F 0 "C?" H 7092 2596 50  0000 L CNN
+F 0 "C17" H 7092 2596 50  0000 L CNN
 F 1 "12p" H 7092 2505 50  0000 L CNN
 F 2 "Capacitor_SMD:C_0402_1005Metric" H 7000 2550 50  0001 C CNN
@@
 $EndComp
 $Comp
-L Device:C_Small C?
+L Device:C_Small C16
 U 1 1 61169E0A
 P 6500 2550
-F 0 "C?" H 6592 2596 50  0000 L CNN
+F 0 "C16" H 6592 2596 50  0000 L CNN
 F 1 "12p" H 6592 2505 50  0000 L CNN
 F 2 "Capacitor_SMD:C_0402_1005Metric" H 6500 2550 50  0001 C CNN
@@
 $EndComp
 $Comp
-L Device:Crystal_GND24_Small Y?
+L Device:Crystal_GND24_Small Y1
 U 1 1 61169E11
 P 6800 2250
-F 0 "Y?" H 6400 2600 50  0000 L CNN
+F 0 "Y1" H 6400 2600 50  0000 L CNN
 F 1 "16MHz" H 6400 2500 50  0000 L CNN
 F 2 "Crystal:Crystal_SMD_3225-4Pin_3.2x2.5mm" H 6800 2250 50  0001 C CNN
@@
 $EndComp
 $Comp
-L Device:LED D?
+L Device:LED D1
 U 1 1 61169E18
 P 4250 3350
-F 0 "D?" H 4243 3095 50  0000 C CNN
+F 0 "D1" H 4243 3095 50  0000 C CNN
 F 1 "LED" H 4243 3186 50  0000 C CNN
 F 2 "LED_SMD:LED_0603_1608Metric" H 4250 3350 50  0001 C CNN
@@
 $EndComp
 $Comp
-L Device:R_Small R?
+L Device:R_Small R1
 U 1 1 61169E1F
 P 4000 3350
-F 0 "R?" V 3804 3350 50  0000 C CNN
+F 0 "R1" V 3804 3350 50  0000 C CNN
 F 1 "1k5" V 3895 3350 50  0000 C CNN
 F 2 "Resistor_SMD:R_0402_1005Metric" H 4000 3350 50  0001 C CNN
@@
 $EndComp
 $Comp
-L Device:C_Small C?
+L Device:C_Small C9
 U 1 1 61169E26
 P 3400 2450
-F 0 "C?" H 3492 2496 50  0000 L CNN
+F 0 "C9" H 3492 2496 50  0000 L CNN
 F 1 "4u7" H 3492 2405 50  0000 L CNN
 F 2 "Capacitor_SMD:C_1206_3216Metric" H 3400 2450 50  0001 C CNN
@@
 $EndComp
 $Comp
-L Device:C_Small C?
+L Device:C_Small C10
 U 1 1 61169E2D
 P 3900 2450
-F 0 "C?" H 3992 2496 50  0000 L CNN
+F 0 "C10" H 3992 2496 50  0000 L CNN
 F 1 "100n" H 3992 2405 50  0000 L CNN
 F 2 "Capacitor_SMD:C_0603_1608Metric" H 3900 2450 50  0001 C CNN
@@
 NoConn ~ 4550 3650
 $Comp
-L JLC_assembled:STM32G030C8T6 U?
+L JLC_assembled:STM32G030C8T6 U6
 U 1 1 61169E68
 P 5300 4750
-F 0 "U?" H 5300 6375 50  0000 C CNN
+F 0 "U6" H 5300 6375 50  0000 C CNN
 F 1 "STM32G030C8T6" H 5300 6284 50  0000 C CNN
-F 2 "" H 5550 7000 50  0001 C CNN
+F 2 "Package_QFP:LQFP-48_7x7mm_P0.5mm" H 5550 7000 50  0001 C CNN
 F 3 "" H 5550 7000 50  0001 C CNN
 	1    5300 4750
@@
 Text HLabel 6050 4650 2    50   Input ~ 0
 SWCLK
-Text HLabel 6050 3750 2    50   Input ~ 0
-DBG_TX
-Text HLabel 6050 4050 2    50   Input ~ 0
-DBG_RX
 Text HLabel 6050 3350 2    50   Input ~ 0
 PB13
@@
 Text HLabel 6050 5700 2    50   Input ~ 0
 PB5
-Text HLabel 6050 5800 2    50   Input ~ 0
-PB6
-Text HLabel 6050 5900 2    50   Input ~ 0
-PB7
 Text HLabel 6050 6000 2    50   Input ~ 0
 PB8
@@
 P 4650 2450
 AR Path="/61169E3B" Ref="C?"  Part="1"
-AR Path="/6116447D/61169E3B" Ref="C?"  Part="1"
-F 0 "C?" H 4742 2496 50  0000 L CNN
+AR Path="/6116447D/61169E3B" Ref="C12"  Part="1"
+F 0 "C12" H 4742 2496 50  0000 L CNN
 F 1 "100n" H 4742 2405 50  0000 L CNN
 F 2 "Capacitor_SMD:C_0603_1608Metric" H 4650 2450 50  0001 C CNN
@@
 P 4300 2450
 AR Path="/61169E34" Ref="C?"  Part="1"
-AR Path="/6116447D/61169E34" Ref="C?"  Part="1"
-F 0 "C?" H 4392 2496 50  0000 L CNN
+AR Path="/6116447D/61169E34" Ref="C11"  Part="1"
+F 0 "C11" H 4392 2496 50  0000 L CNN
 F 1 "100n" H 4392 2405 50  0000 L CNN
 F 2 "Capacitor_SMD:C_0603_1608Metric" H 4300 2450 50  0001 C CNN
@@
 P 5000 2450
 AR Path="/61175BE9" Ref="C?"  Part="1"
-AR Path="/6116447D/61175BE9" Ref="C?"  Part="1"
-F 0 "C?" H 5092 2496 50  0000 L CNN
+AR Path="/6116447D/61175BE9" Ref="C13"  Part="1"
+F 0 "C13" H 5092 2496 50  0000 L CNN
 F 1 "100n" H 5092 2405 50  0000 L CNN
 F 2 "Capacitor_SMD:C_0603_1608Metric" H 5000 2450 50  0001 C CNN
@@
 P 5350 2450
 AR Path="/611762EE" Ref="C?"  Part="1"
-AR Path="/6116447D/611762EE" Ref="C?"  Part="1"
-F 0 "C?" H 5442 2496 50  0000 L CNN
+AR Path="/6116447D/611762EE" Ref="C14"  Part="1"
+F 0 "C14" H 5442 2496 50  0000 L CNN
 F 1 "100n" H 5442 2405 50  0000 L CNN
 F 2 "Capacitor_SMD:C_0603_1608Metric" H 5350 2450 50  0001 C CNN
@@
 P 5700 2450
 AR Path="/61176759" Ref="C?"  Part="1"
-AR Path="/6116447D/61176759" Ref="C?"  Part="1"
-F 0 "C?" H 5792 2496 50  0000 L CNN
+AR Path="/6116447D/61176759" Ref="C15"  Part="1"
+F 0 "C15" H 5792 2496 50  0000 L CNN
 F 1 "100n" H 5792 2405 50  0000 L CNN
 F 2 "Capacitor_SMD:C_0603_1608Metric" H 5700 2450 50  0001 C CNN
@@
 Wire Wire Line
 	5350 2350 5000 2350
+Text HLabel 6050 3750 2    50   Input ~ 0
+PA9
+Text HLabel 6050 4050 2    50   Input ~ 0
+PA10
+Text HLabel 6050 5900 2    50   Input ~ 0
+PB7
+Text HLabel 6050 5800 2    50   Input ~ 0
+PB6
 $EndSCHEMATC

Commit message: Lora-module v1
Parts:
- U6: symbol JLC_assembled:STM32G030C8T6 -> jantteri-lora-rescue:STM32G030C8T6-JLC_assembled; LCSC (none) -> C529329
Changed lines of the file:
@@
 $Descr A4 11693 8268
 encoding utf-8
-Sheet 3 8
+Sheet 8 8
 Title ""
 Date ""
@@
 NoConn ~ 4550 3650
 $Comp
-L JLC_assembled:STM32G030C8T6 U6
+L jantteri-lora-rescue:STM32G030C8T6-JLC_assembled U6
 U 1 1 61169E68
 P 5300 4750
@@
 F 2 "Package_QFP:LQFP-48_7x7mm_P0.5mm" H 5550 7000 50  0001 C CNN
 F 3 "" H 5550 7000 50  0001 C CNN
+F 4 "C529329" H 5300 4750 50  0001 C CNN "LCSC"
 	1    5300 4750
 	1    0    0    -1
