File: jantteri-hit-detector/led-strip-ctrl.sch (KiCad schematic (older format))
At the start: 5 parts, among them J4 Conn_01x04_Male, U8 TXB0104RUT

Commit message: random changes
Parts:
- U8: LCSC (none) -> C105266
Changed lines of the file:
@@
 $Descr A4 11693 8268
 encoding utf-8
-Sheet 11 11
+Sheet 8 11
 Title ""
 Date ""
@@
 F 2 "Package_DFN_QFN:Texas_R_PUQFN-N12" H 4800 2900 50  0001 C CNN
 F 3 "http://www.ti.com/lit/ds/symlink/txb0104.pdf" H 4910 3745 50  0001 C CNN
+F 4 " C105266 " H 4800 3650 50  0001 C CNN "LCSC"
 	1    4800 3650
 	1    0    0    -1
