File: jantteri-hit-detector/LIS2DW12.sch (KiCad schematic (older format))
At the start: 3 parts, among them U3 LIS2DW12TR

Commit message: Tuubijantteri design Ordered
Changed lines of the file:
@@
 $Descr A4 11693 8268
 encoding utf-8
-Sheet 9 11
+Sheet 6 7
 Title ""
 Date ""
@@
 AR Path="/615681DE/611ECB68" Ref="C14"  Part="1"
 AR Path="/6156935E/611ECB68" Ref="C16"  Part="1"
-F 0 "C12" V 4200 2850 50  0000 L CNN
+F 0 "C16" V 4200 2850 50  0000 L CNN
 F 1 "100n" V 4100 2800 50  0000 L CNN
 F 2 "Capacitor_SMD:C_0603_1608Metric" H 4350 2900 50  0001 C CNN
@@
 AR Path="/615681DE/611ECB6F" Ref="C15"  Part="1"
 AR Path="/6156935E/611ECB6F" Ref="C17"  Part="1"
-F 0 "C13" V 4950 2850 50  0000 L CNN
+F 0 "C17" V 4950 2850 50  0000 L CNN
 F 1 "100n" V 5050 2800 50  0000 L CNN
 F 2 "Capacitor_SMD:C_0603_1608Metric" H 4800 2900 50  0001 C CNN
@@
 AR Path="/615681DE/6155FBE2" Ref="U4"  Part="1"
 AR Path="/6156935E/6155FBE2" Ref="U5"  Part="1"
-F 0 "U3" H 5050 4500 50  0000 L CNN
+F 0 "U5" H 5050 4500 50  0000 L CNN
 F 1 "LIS2DW12TR" H 5000 4400 50  0000 L CNN
 F 2 "Package_LGA:LGA-12_2x2mm_P0.5mm" H 4800 2850 50  0001 C CNN
