File: jantteri-motor-pwr/power_protect.sch (KiCad schematic (older format))
At the start: 5 parts, among them Q1 IRLML6402TRPBF, U2 AP2301

Commit message: jantteri-pwr-motor
Parts:
- renumbered Q1 to Q2, R3 to R5, U2 to U3
Changed lines of the file:
@@
 $Descr A4 11693 8268
 encoding utf-8
-Sheet 9 11
+Sheet 4 10
 Title ""
 Date ""
@@
 AR Path="/611A8D7A/61181872" Ref="C?"  Part="1"
 AR Path="/611E498E/61181872" Ref="C10"  Part="1"
-AR Path="/612244CD/61181872" Ref="C20"  Part="1"
-F 0 "C20" H 4342 2946 50  0000 L CNN
+AR Path="/612244CD/61181872" Ref="C14"  Part="1"
+F 0 "C10" H 4342 2946 50  0000 L CNN
 F 1 "100n" H 4342 2855 50  0000 L CNN
 F 2 "Capacitor_SMD:C_0603_1608Metric" H 4250 2900 50  0001 C CNN
@@
 AR Path="/611A8D7A/61186B4B" Ref="C?"  Part="1"
 AR Path="/611E498E/61186B4B" Ref="C11"  Part="1"
-AR Path="/612244CD/61186B4B" Ref="C21"  Part="1"
-F 0 "C21" H 5992 2946 50  0000 L CNN
+AR Path="/612244CD/61186B4B" Ref="C15"  Part="1"
+F 0 "C11" H 5992 2946 50  0000 L CNN
 F 1 "100n" H 5992 2855 50  0000 L CNN
 F 2 "Capacitor_SMD:C_0603_1608Metric" H 5900 2900 50  0001 C CNN
@@
 AR Path="/6117A90D/611A29C1" Ref="Q?"  Part="1"
 AR Path="/611A8D7A/611A29C1" Ref="Q?"  Part="1"
-AR Path="/611E498E/611A29C1" Ref="Q1"  Part="1"
-AR Path="/612244CD/611A29C1" Ref="Q2"  Part="1"
+AR Path="/611E498E/611A29C1" Ref="Q2"  Part="1"
+AR Path="/612244CD/611A29C1" Ref="Q3"  Part="1"
 F 0 "Q2" V 4042 2900 50  0000 C CNN
 F 1 "IRLML6402TRPBF" V 3951 2900 50  0000 C CNN
@@
 AR Path="/6117A90D/611A520B" Ref="R?"  Part="1"
 AR Path="/611A8D7A/611A520B" Ref="R?"  Part="1"
-AR Path="/611E498E/611A520B" Ref="R3"  Part="1"
-AR Path="/612244CD/611A520B" Ref="R4"  Part="1"
-F 0 "R4" H 4659 3396 50  0000 L CNN
+AR Path="/611E498E/611A520B" Ref="R5"  Part="1"
+AR Path="/612244CD/611A520B" Ref="R6"  Part="1"
+F 0 "R5" H 4659 3396 50  0000 L CNN
 F 1 "100K" H 4659 3305 50  0000 L CNN
 F 2 "Resistor_SMD:R_0402_1005Metric" H 4600 3350 50  0001 C CNN
@@
 	5000 3450 5000 3250
 $Comp
-L JLC_assembled:AP2301 U2
+L JLC_assembled:AP2301 U3
 U 1 1 611E51A5
 P 4950 2900
-AR Path="/611E498E/611E51A5" Ref="U2"  Part="1"
-AR Path="/612244CD/611E51A5" Ref="U7"  Part="1"
-F 0 "U7" H 5000 3465 50  0000 C CNN
+AR Path="/611E498E/611E51A5" Ref="U3"  Part="1"
+AR Path="/612244CD/611E51A5" Ref="U5"  Part="1"
+F 0 "U3" H 5000 3465 50  0000 C CNN
 F 1 "AP2301" H 5000 3374 50  0000 C CNN
 F 2 "Package_SO:MSOP-8-1EP_3x3mm_P0.65mm_EP1.68x1.88mm" H 5150 2500 50  0001 C CNN

Commit message: revised motor-pwr
Parts:
- U3: symbol JLC_assembled:AP2301 -> jantteri-motor-pwr-rescue:AP2301-JLC_assembled
Changed lines of the file:
@@
 $Descr A4 11693 8268
 encoding utf-8
-Sheet 4 10
+Sheet 6 10
 Title ""
 Date ""
@@
 AR Path="/611E498E/61181872" Ref="C10"  Part="1"
 AR Path="/612244CD/61181872" Ref="C14"  Part="1"
-F 0 "C10" H 4342 2946 50  0000 L CNN
+F 0 "C14" H 4342 2946 50  0000 L CNN
 F 1 "100n" H 4342 2855 50  0000 L CNN
 F 2 "Capacitor_SMD:C_0603_1608Metric" H 4250 2900 50  0001 C CNN
@@
 AR Path="/611E498E/61186B4B" Ref="C11"  Part="1"
 AR Path="/612244CD/61186B4B" Ref="C15"  Part="1"
-F 0 "C11" H 5992 2946 50  0000 L CNN
+F 0 "C15" H 5992 2946 50  0000 L CNN
 F 1 "100n" H 5992 2855 50  0000 L CNN
 F 2 "Capacitor_SMD:C_0603_1608Metric" H 5900 2900 50  0001 C CNN
@@
 AR Path="/611E498E/611A29C1" Ref="Q2"  Part="1"
 AR Path="/612244CD/611A29C1" Ref="Q3"  Part="1"
-F 0 "Q2" V 4042 2900 50  0000 C CNN
+F 0 "Q3" V 4042 2900 50  0000 C CNN
 F 1 "IRLML6402TRPBF" V 3951 2900 50  0000 C CNN
 F 2 "Package_TO_SOT_SMD:SOT-23" H 3900 2825 50  0001 L CIN
@@
 AR Path="/611E498E/611A520B" Ref="R5"  Part="1"
 AR Path="/612244CD/611A520B" Ref="R6"  Part="1"
-F 0 "R5" H 4659 3396 50  0000 L CNN
+F 0 "R6" H 4659 3396 50  0000 L CNN
 F 1 "100K" H 4659 3305 50  0000 L CNN
 F 2 "Resistor_SMD:R_0402_1005Metric" H 4600 3350 50  0001 C CNN
@@
 	5000 3450 5000 3250
 $Comp
-L JLC_assembled:AP2301 U3
+L jantteri-motor-pwr-rescue:AP2301-JLC_assembled U3
 U 1 1 611E51A5
 P 4950 2900
 AR Path="/611E498E/611E51A5" Ref="U3"  Part="1"
 AR Path="/612244CD/611E51A5" Ref="U5"  Part="1"
-F 0 "U3" H 5000 3465 50  0000 C CNN
+AR Path="/611E51A5" Ref="U3"  Part="1"
+F 0 "U5" H 5000 3465 50  0000 C CNN
 F 1 "AP2301" H 5000 3374 50  0000 C CNN
 F 2 "Package_SO:MSOP-8-1EP_3x3mm_P0.65mm_EP1.68x1.88mm" H 5150 2500 50  0001 C CNN

Commit message: random changes
Changed lines of the file:
@@
 $Descr A4 11693 8268
 encoding utf-8
-Sheet 6 10
+Sheet 4 10
 Title ""
 Date ""
@@
 AR Path="/611E498E/61181872" Ref="C10"  Part="1"
 AR Path="/612244CD/61181872" Ref="C14"  Part="1"
-F 0 "C14" H 4342 2946 50  0000 L CNN
+F 0 "C10" H 4342 2946 50  0000 L CNN
 F 1 "100n" H 4342 2855 50  0000 L CNN
 F 2 "Capacitor_SMD:C_0603_1608Metric" H 4250 2900 50  0001 C CNN
@@
 AR Path="/611E498E/61186B4B" Ref="C11"  Part="1"
 AR Path="/612244CD/61186B4B" Ref="C15"  Part="1"
-F 0 "C15" H 5992 2946 50  0000 L CNN
+F 0 "C11" H 5992 2946 50  0000 L CNN
 F 1 "100n" H 5992 2855 50  0000 L CNN
 F 2 "Capacitor_SMD:C_0603_1608Metric" H 5900 2900 50  0001 C CNN
@@
 AR Path="/611E498E/611A29C1" Ref="Q2"  Part="1"
 AR Path="/612244CD/611A29C1" Ref="Q3"  Part="1"
-F 0 "Q3" V 4042 2900 50  0000 C CNN
+F 0 "Q2" V 4042 2900 50  0000 C CNN
 F 1 "IRLML6402TRPBF" V 3951 2900 50  0000 C CNN
 F 2 "Package_TO_SOT_SMD:SOT-23" H 3900 2825 50  0001 L CIN
@@
 AR Path="/611E498E/611A520B" Ref="R5"  Part="1"
 AR Path="/612244CD/611A520B" Ref="R6"  Part="1"
-F 0 "R6" H 4659 3396 50  0000 L CNN
+F 0 "R5" H 4659 3396 50  0000 L CNN
 F 1 "100K" H 4659 3305 50  0000 L CNN
 F 2 "Resistor_SMD:R_0402_1005Metric" H 4600 3350 50  0001 C CNN
@@
 AR Path="/612244CD/611E51A5" Ref="U5"  Part="1"
 AR Path="/611E51A5" Ref="U3"  Part="1"
-F 0 "U5" H 5000 3465 50  0000 C CNN
+F 0 "U3" H 5000 3465 50  0000 C CNN
 F 1 "AP2301" H 5000 3374 50  0000 C CNN
 F 2 "Package_SO:MSOP-8-1EP_3x3mm_P0.65mm_EP1.68x1.88mm" H 5150 2500 50  0001 C CNN
