File: jantteri-motor-pwr/10pinARM.sch (KiCad schematic (older format))
At the start: 1 part

Commit message: jantteri-pwr-motor
Parts:
- J2: renamed from J?; footprint Connector_PinHeader_1.27mm:PinHeader_2x05_P1.27mm_Vertical_SMD -> Connector_PinHeader_1.27mm:PinHeader_2x05_P1.27mm_Horizontal
Changed lines of the file:
@@
 $Descr A4 11693 8268
 encoding utf-8
-Sheet 4 8
+Sheet 3 10
 Title ""
 Date ""
@@
 	5000 3400 4900 3400
 $Comp
-L Connector_Generic:Conn_02x05_Odd_Even J?
+L Connector_Generic:Conn_02x05_Odd_Even J2
 U 1 1 6115169A
 P 5200 3600
-AR Path="/6115169A" Ref="J?"  Part="1"
-AR Path="/61150666/6115169A" Ref="J?"  Part="1"
-F 0 "J?" H 5250 4017 50  0000 C CNN
+F 0 "J2" H 5250 4017 50  0000 C CNN
 F 1 "SWD" H 5250 3926 50  0000 C CNN
-F 2 "Connector_PinHeader_1.27mm:PinHeader_2x05_P1.27mm_Vertical_SMD" H 5200 3600 50  0001 C CNN
+F 2 "Connector_PinHeader_1.27mm:PinHeader_2x05_P1.27mm_Horizontal" H 5200 3600 50  0001 C CNN
 F 3 "~" H 5200 3600 50  0001 C CNN
 	1    5200 3600
