File: tuubijantteri/jantteri_right/_autosave-jantteri_right.kicad_pcb (KiCad board)
At the start: 2 copper layers, 63.8 x 63.8 mm, 83 parts, among them J1 USB_C_Receptacle_USB2.0, J2 Conn_01x02_Male, J3 Conn_01x02_Male, J4 Conn_02x08_Odd_Even, Q1 AP3407, Q2 AP3404S, Q3 AP3404S, Q4 AP3404S, Q5 AP3407, U1 STUSB4500QTR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

Commit message: Update jantteri-right to new layout
Other:
- board text added: "B+"
- board text added: "B-"
- board text added: "GND"
- board text added: "M+"
- board text added: "M-"
- board text added: "VOUT"
Changed lines of the file:
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@@
   (general
     (thickness 1.6)
-    (drawings 26)
+    (drawings 32)
     (tracks 810)
     (zones 0)
@@
   (page A4)
   (layers
-    (0 F.Cu signal)
-    (31 B.Cu signal hide)
+    (0 F.Cu signal hide)
+    (31 B.Cu signal)
     (32 B.Adhes user hide)
     (33 F.Adhes user hide)
     (34 B.Paste user hide)
     (35 F.Paste user hide)
-    (36 B.SilkS user hide)
+    (36 B.SilkS user)
     (37 F.SilkS user)
     (38 B.Mask user hide)
@@
     (44 Edge.Cuts user)
     (45 Margin user hide)
-    (46 B.CrtYd user hide)
+    (46 B.CrtYd user)
     (47 F.CrtYd user)
     (48 B.Fab user hide)
@@
     )
   )
+  (gr_text B- (at 158.23438 86.35746) (layer B.SilkS)
+    (effects (font (size 1 1) (thickness 0.15)) (justify mirror))
+  )
+  (gr_text B+ (at 168.76014 86.9442) (layer B.SilkS)
+    (effects (font (size 1 1) (thickness 0.15)) (justify mirror))
+  )
+  (gr_text M- (at 116.1923 74.90714) (layer B.SilkS)
+    (effects (font (size 1 1) (thickness 0.15)) (justify mirror))
+  )
+  (gr_text M+ (at 115.7097 85.4583) (layer B.SilkS)
+    (effects (font (size 1 1) (thickness 0.15)) (justify mirror))
+  )
+  (gr_text GND (at 118.01094 87.2363) (layer B.SilkS)
+    (effects (font (size 1 1) (thickness 0.15)) (justify mirror))
+  )
+  (gr_text VOUT (at 111.71682 87.06104) (layer B.SilkS)
+    (effects (font (size 1 1) (thickness 0.15)) (justify mirror))
+  )
   (target plus (at 139.2174 85.2297) (size 5) (width 0.05) (layer Edge.Cuts))
