File: tuubijantteri/jantteri_right/DRV8848.sch (KiCad schematic (older format))
At the start: 4 parts, among them U2 DRV8848

Commit message: update jantteri_right
Parts:
- C12: LCSC C49217 -> C377773
Changed lines of the file:
@@
 F 2 "Capacitor_SMD:C_0805_2012Metric" H 6250 3300 50  0001 C CNN
 F 3 "~" H 6250 3300 50  0001 C CNN
-F 4 "C49217" H 6250 3300 50  0001 C CNN "LCSC"
+F 4 "C377773" H 6250 3300 50  0001 C CNN "LCSC"
 	1    6250 3300
 	1    0    0    -1
