File: tuubijantteri/jantteri_right/jantteri_right.sch (KiCad schematic (older format))
At the start: 3 parts, among them J2 Conn_01x02_Male, J3 Conn_01x02_Male, J4 Conn_02x08_Odd_Even

Commit message: update jantteri_right
Parts:
- J2, J3: LCSC (none) -> C160315
- J4: LCSC (none) -> C178295
Changed lines of the file:
@@
 F 2 "Connector_JST2:JST_VH_B2P-VH-B_1x02_P3.96mm_Vertical" H 4600 1600 50  0001 C CNN
 F 3 "~" H 4600 1600 50  0001 C CNN
+F 4 "C160315" H 4600 1600 50  0001 C CNN "LCSC"
 	1    4600 1600
 	-1   0    0    1
@@
 F 2 "Connector_JST2:JST_VH_B2P-VH-B_1x02_P3.96mm_Vertical" H 5500 2550 50  0001 C CNN
 F 3 "~" H 5500 2550 50  0001 C CNN
+F 4 "C160315" H 5500 2550 50  0001 C CNN "LCSC"
 	1    5500 2550
 	1    0    0    -1
@@
 F 2 "Connector_PinHeader_1.27mm:PinHeader_2x08_P1.27mm_Vertical_SMD" H 9500 2900 50  0001 C CNN
 F 3 "~" H 9500 2900 50  0001 C CNN
+F 4 "C178295" H 9500 2900 50  0001 C CNN "LCSC"
 	1    9500 2900
 	1    0    0    -1
@@
 DRV_n_FAULT_out
 $Comp
-L power:GND #PWR?
+L power:GND #PWR0104
 U 1 1 66054A37
 P 9300 2700
-F 0 "#PWR?" H 9300 2450 50  0001 C CNN
+F 0 "#PWR0104" H 9300 2450 50  0001 C CNN
 F 1 "GND" V 9305 2572 50  0000 R CNN
 F 2 "" H 9300 2700 50  0001 C CNN
