File: tuubijantteri/jantteri_right/usbc.sch (KiCad schematic (older format))
At the start: 23 parts, among them J1 USB_C_Receptacle_USB2.0, Q5 AP3407, U1 STUSB4500QTR

Commit message: tuubijantteri order changes
Parts:
- D6: LCSC C309871 -> C123807
Changed lines of the file:
@@
 F 2 "Diode_SMD:D_SOD-123F" H 4300 1900 50  0001 C CNN
 F 3 "~" H 4300 1900 50  0001 C CNN
-F 4 "C309871" V 4300 1900 50  0001 C CNN "LCSC"
+F 4 "C123807" V 4300 1900 50  0001 C CNN "LCSC"
 	1    4300 1900
 	0    1    1    0
