File: tuubijantteri/jantteri_left/5V-buck.sch (KiCad schematic (older format))
At the start: 5 parts, among them U3 LM2596S-5

Commit message: update jantteri_right
Parts:
- C16: LCSC C171665 -> C8024
Changed lines of the file:
@@
 $Descr A4 11693 8268
 encoding utf-8
-Sheet 8 10
+Sheet 7 10
 Title ""
 Date ""
@@
 F 2 "Capacitor_Tantalum_SMD:CP_EIA-7343-31_Kemet-D" H 5950 3200 50  0001 C CNN
 F 3 "~" H 5950 3200 50  0001 C CNN
-F 4 " C171665" H 5950 3200 50  0001 C CNN "LCSC"
+F 4 " C8024" H 5950 3200 50  0001 C CNN "LCSC"
 	1    5950 3200
 	1    0    0    -1
