File: tuubijantteri/jantteri_left/STM32L151C8T6A.sch (KiCad schematic (older format))
At the start: 18 parts, among them U2 STM32L151C8TxA, Y1 16MHz

Commit message: update jantteri_right
Parts:
- D1: LCSC C72041 -> C2286
Changed lines of the file:
@@
 F 2 "LED_SMD:LED_0603_1608Metric" H 3950 4750 50  0001 C CNN
 F 3 "~" H 3950 4750 50  0001 C CNN
-F 4 "C72041" H 3950 4750 50  0001 C CNN "LCSC"
+F 4 "C2286" H 3950 4750 50  0001 C CNN "LCSC"
 	1    3950 4750
 	1    0    0    -1
