File: tuubijantteri/jantteri_left/jantteri_left.sch (KiCad schematic (older format))
At the start: 11 parts, among them J1 Conn_02x08_Odd_Even, J2 Conn_01x03_Male, Q1 AO3400A, SW1 SW_Push

Commit message: update jantteri_right
Parts:
- J1: LCSC (none) -> C178295
- SW1: value SW_Push -> TS-1095PS-A11B3-C3D2
Changed lines of the file:
@@
 F 2 "Connector_PinHeader_1.27mm:PinHeader_2x08_P1.27mm_Vertical_SMD" H 1450 1200 50  0001 C CNN
 F 3 "~" H 1450 1200 50  0001 C CNN
+F 4 "C178295" H 1450 1200 50  0001 C CNN "LCSC"
 	1    1450 1200
 	1    0    0    -1
@@
 P 5250 1650
 F 0 "SW1" H 5250 1935 50  0000 C CNN
-F 1 "SW_Push" H 5250 1844 50  0000 C CNN
+F 1 "TS-1095PS-A11B3-C3D2" H 5250 1844 50  0000 C CNN
 F 2 "voja-footprints:TS-1095PS-A11B3-C3D2" H 5250 1850 50  0001 C CNN
 F 3 "https://wmsc.lcsc.com/wmsc/upload/file/pdf/v2/lcsc/2304140030_Yuandi-TS-1095PS-A11B3-C3D2_C2834951.pdf" H 5250 1850 50  0001 C CNN
